Commit message: Test for visual servoing

File: src/baxter_common/baxter_description/urdf/pedestal/pedestal.xacro (robot description, xacro)
@@ -36,5 +36,5 @@
       <parent link="world"/>
       <child link="base"/>
-      <origin xyz="0 1 0.93" rpy="0 0 -1.57079632679" />
+      <!--origin xyz="0 1 0.93" rpy="0 0 0" /-->
     </joint>
   <!--/xacro:if-->
